Commit message: Rotate bilateral hand and wrist-camera mounts around forearm axis

File: assets/assembly_bilateral_axis180.urdf (robot description, URDF)
Before this commit: robot tron2_dach_revo3_d455_supplied_step_brackets, 116 links, 115 joints
Joints:
- joint world_to_base: origin xyz=0 0 1.2 rpy=0 0 0 -> xyz=0 0 1.20035 rpy=0 0 0
