Commit message: Rotate hands and wrist cameras 180 degrees

File: assets/assembly.urdf (robot description, URDF)
Before this commit: robot tron2_dach_revo3_d455_supplied_step_brackets, 116 links, 115 joints
Joints:
- joint left_hand_base_joint: origin xyz=0 0.023855 0 rpy=-1.57079632679 1.57079632679 0 -> xyz=0 0.023855 0 rpy=-1.57079632679 -1.57079632679 0
- joint left_wrist_camera_reference_joint: origin xyz=-0.0317 -1.31006316906e-18 -0.0753 rpy=1.57079632679 0 1.57079632679 -> xyz=-0.0317 -1.31006316906e-18 -0.0753 rpy=-1.57079632679 0 -1.57079632679
- joint right_hand_base_joint: origin xyz=0 0.023855 0 rpy=-1.57079632679 -1.57079632679 0 -> xyz=0 0.023855 0 rpy=-1.57079632679 1.57079632679 0
- joint right_wrist_camera_reference_joint: origin xyz=-0.0317 -1.31006316906e-18 -0.0753 rpy=1.57079632679 2.22044604925e-16 -1.57079632679 -> xyz=-0.0317 -1.31006316906e-18 -0.0753 rpy=-1.57079632679 0 1.57079632679

Commit message: Fix wrist camera 180 degree orbit

File: assets/assembly.urdf (robot description, URDF)
Before this commit: robot tron2_dach_revo3_d455_supplied_step_brackets, 116 links, 115 joints
Joints:
- joint left_wrist_camera_reference_joint: origin xyz=-0.0317 -1.31006316906e-18 -0.0753 rpy=-1.57079632679 0 -1.57079632679 -> xyz=-0.0317 0 0.0753 rpy=-1.57079632679 0 -1.57079632679
- joint right_wrist_camera_reference_joint: origin xyz=-0.0317 -1.31006316906e-18 -0.0753 rpy=-1.57079632679 0 1.57079632679 -> xyz=-0.0317 0 0.0753 rpy=-1.57079632679 0 1.57079632679

Commit message: Replace head camera with D455 and update colors

File: assets/assembly.urdf (robot description, URDF)
Before this commit: robot tron2_dach_revo3_supplied_step_brackets, 107 links, 106 joints
Links:
- added link head_camera_accel_frame
- added link head_camera_accel_optical_frame
- added link head_camera_gyro_frame
- added link head_camera_gyro_optical_frame
- added link head_camera_imu_optical_frame
- added link head_camera_infra1_frame
- added link head_camera_infra1_optical_frame
- added link head_camera_infra2_frame
- added link head_camera_infra2_optical_frame
- link base_Link: geometry collision mesh filename=meshes/tron2/base_Link.STL; visual box size=0.006 0.050 0.070
- link head_camera_link: mass None -> 0.072; geometry collision box size=0.026 0.124 0.029; visual mesh filename=meshes/cameras/d455_visual_mm.stl scale=0.001 0.001 0.001
- link proximal_yaw_L_Link: geometry collision mesh filename=meshes/tron2/proximal_yaw_L_Link_collision.STL; visual cylinder length=0.010 radius=0.054
- link proximal_yaw_R_Link: geometry collision mesh filename=meshes/tron2/proximal_yaw_R_Link_collision.STL; visual cylinder length=0.010 radius=0.054
- link wrist_yaw_L_Link: geometry collision mesh filename=meshes/tron2/wrist_yaw_L_Link.STL; visual cylinder length=0.008 radius=0.043
- link wrist_yaw_R_Link: geometry collision mesh filename=meshes/tron2/wrist_yaw_R_Link.STL; visual cylinder length=0.008 radius=0.043
Joints:
- added joint head_camera_accel_joint: type fixed, parent head_camera_link, child head_camera_accel_frame, origin xyz=-0.01602 -0.03022 0.0074 rpy=0 0 0
- added joint head_camera_accel_optical_joint: type fixed, parent head_camera_accel_frame, child head_camera_accel_optical_frame, origin xyz=0 0 0 rpy=-1.57079632679 0 -1.57079632679
- added joint head_camera_gyro_joint: type fixed, parent head_camera_link, child head_camera_gyro_frame, origin xyz=-0.01602 -0.03022 0.0074 rpy=0 0 0
- added joint head_camera_gyro_optical_joint: type fixed, parent head_camera_gyro_frame, child head_camera_gyro_optical_frame, origin xyz=0 0 0 rpy=-1.57079632679 0 -1.57079632679
- added joint head_camera_imu_optical_joint: type fixed, parent head_camera_gyro_optical_frame, child head_camera_imu_optical_frame, origin xyz=0 0 0 rpy=0 0 0
- added joint head_camera_infra1_joint: type fixed, parent head_camera_link, child head_camera_infra1_frame, origin xyz=0 0 0 rpy=0 0 0
- added joint head_camera_infra1_optical_joint: type fixed, parent head_camera_infra1_frame, child head_camera_infra1_optical_frame, origin xyz=0 0 0 rpy=-1.57079632679 0 -1.57079632679
- added joint head_camera_infra2_joint: type fixed, parent head_camera_link, child head_camera_infra2_frame, origin xyz=0 -0.095 0 rpy=0 0 0
- added joint head_camera_infra2_optical_joint: type fixed, parent head_camera_infra2_frame, child head_camera_infra2_optical_frame, origin xyz=0 0 0 rpy=-1.57079632679 0 -1.57079632679
- joint head_camera_color_joint: origin xyz=0 0.015 0 rpy=0 0 0 -> xyz=0 -0.059 0 rpy=0 0 0
- joint head_camera_link_joint: origin xyz=0.0106 0.0175 0.0125 rpy=0 0 0 -> xyz=0.01115 0.0475 0.0145 rpy=0 0 0

Commit message: Rotate wrist camera brackets about finger axis

File: assets/assembly.urdf (robot description, URDF)
Before this commit: robot tron2_dach_revo3_d455_supplied_step_brackets, 116 links, 115 joints
Joints:
- joint left_wrist_camera_reference_joint: origin xyz=-0.0317 -1.31006316906e-18 -0.0753 rpy=1.57079632679 0 1.57079632679 -> xyz=-0.0317 -1.31006316906e-18 -0.0753 rpy=1.57079632679 0 -1.57079632679
- joint right_wrist_camera_reference_joint: origin xyz=-0.0317 -1.31006316906e-18 -0.0753 rpy=1.57079632679 2.22044604925e-16 -1.57079632679 -> xyz=-0.0317 -1.31006316906e-18 -0.0753 rpy=1.57079632679 0 1.57079632679

Commit message: Restore original wrist camera transforms

File: assets/assembly.urdf (robot description, URDF)
Before this commit: robot tron2_dach_revo3_d455_supplied_step_brackets, 116 links, 115 joints
Joints:
- joint left_wrist_camera_reference_joint: origin xyz=-0.0317 0 0.0753 rpy=1.57079632679 0 1.57079632679 -> xyz=-0.0317 -1.31006316906e-18 -0.0753 rpy=1.57079632679 0 1.57079632679
- joint right_wrist_camera_reference_joint: origin xyz=-0.0317 0 0.0753 rpy=1.57079632679 2.22044604925e-16 -1.57079632679 -> xyz=-0.0317 -1.31006316906e-18 -0.0753 rpy=1.57079632679 2.22044604925e-16 -1.57079632679

Commit message: Restore wrist camera attitude at opposite arm side

File: assets/assembly.urdf (robot description, URDF)
Before this commit: robot tron2_dach_revo3_d455_supplied_step_brackets, 116 links, 115 joints
Joints:
- joint left_wrist_camera_reference_joint: origin xyz=-0.0317 0 0.0753 rpy=-1.57079632679 0 -1.57079632679 -> xyz=-0.0317 0 0.0753 rpy=1.57079632679 0 1.57079632679
- joint right_wrist_camera_reference_joint: origin xyz=-0.0317 0 0.0753 rpy=-1.57079632679 0 1.57079632679 -> xyz=-0.0317 0 0.0753 rpy=1.57079632679 2.22044604925e-16 -1.57079632679

Commit message: Set robot origin 45 cm above work table

File: assets/assembly.urdf (robot description, URDF)
Before this commit: robot tron2_dach_revo3_d455_supplied_step_brackets, 116 links, 115 joints
Joints:
- joint world_to_base: origin xyz=0 0 1.20035 rpy=0 0 0 -> xyz=0 0 1.2 rpy=0 0 0
