Commit message: Migrate Revo3 hands to official kinematics

File: assets/assembly.urdf (robot description, URDF)
Before this commit: robot tron2_dach_revo3_d455_supplied_step_brackets, 116 links, 115 joints
Links:
- removed link left_palm
- removed link right_palm
- link left_hand_base_link: geometry collision mesh filename=meshes/hands/collision/left/left_hand_base_link.STL; collision mesh filename=meshes/hands/collision/left/left_palm_backtrim_v2.obj
- link left_index_DIP_Link: mass 0.008 -> 0.011; geometry collision mesh filename=meshes/hands/collision/left/left_index_DIP_link.STL; collision mesh filename=meshes/hands/collision/left/left_index_DIP_rubber_link.STL
- link left_index_MCP_Link: geometry collision mesh filename=meshes/hands/collision/left/left_index_MCP_link.STL; collision mesh filename=meshes/hands/collision/left/left_index_MCP_rubber_link.STL
- link left_index_MPR_Link: geometry collision mesh filename=meshes/hands/collision/left/left_index_MPR_link.STL; visual mesh filename=meshes/hands/visual/left/left_index_MPR_link.STL
- link left_index_PIP_Link: mass 0.031 -> 0.0332; geometry collision mesh filename=meshes/hands/collision/left/left_index_PIP_link.STL; collision mesh filename=meshes/hands/collision/left/left_index_PIP_rubber_link.STL
- link left_little_DIP_Link: mass 0.01 -> 0.011; geometry collision mesh filename=meshes/hands/collision/left/left_little_DIP_link.STL; collision mesh filename=meshes/hands/collision/left/left_little_DIP_rubber_link.STL
- link left_little_MCP_Link: geometry collision mesh filename=meshes/hands/collision/left/left_little_MCP_link.STL; collision mesh filename=meshes/hands/collision/left/left_little_MCP_rubber_link.STL
- link left_little_MPR_Link: geometry collision mesh filename=meshes/hands/collision/left/left_little_MPR_link.STL; visual mesh filename=meshes/hands/visual/left/left_little_MPR_link.STL
- link left_little_PIP_Link: geometry collision mesh filename=meshes/hands/collision/left/left_little_PIP_link.STL; collision mesh filename=meshes/hands/collision/left/left_little_PIP_rubber_link.STL
- link left_middle_DIP_Link: mass 0.01 -> 0.011; geometry collision mesh filename=meshes/hands/collision/left/left_middle_DIP_link.STL; collision mesh filename=meshes/hands/collision/left/left_middle_DIP_rubber_link.STL
- link left_middle_MCP_Link: geometry collision mesh filename=meshes/hands/collision/left/left_middle_MCP_link.STL; collision mesh filename=meshes/hands/collision/left/left_middle_MCP_rubber_link.STL
- link left_middle_MPR_Link: mass 0.012 -> 0.013; geometry collision mesh filename=meshes/hands/collision/left/left_middle_MPR_link.STL; visual mesh filename=meshes/hands/visual/left/left_middle_MPR_link.STL
- link left_middle_PIP_Link: mass 0.031 -> 0.0332; geometry collision mesh filename=meshes/hands/collision/left/left_middle_PIP_link.STL; collision mesh filename=meshes/hands/collision/left/left_middle_PIP_rubber_link.STL
- link left_ring_DIP_Link: mass 0.01 -> 0.011; geometry collision mesh filename=meshes/hands/collision/left/left_ring_DIP_link.STL; collision mesh filename=meshes/hands/collision/left/left_ring_DIP_rubber_link.STL
- link left_ring_MCP_Link: geometry collision mesh filename=meshes/hands/collision/left/left_ring_MCP_link.STL; collision mesh filename=meshes/hands/collision/left/left_ring_MCP_rubber_link.STL
- link left_ring_MPR_Link: geometry collision mesh filename=meshes/hands/collision/left/left_ring_MPR_link.STL; visual mesh filename=meshes/hands/visual/left/left_ring_MPR_link.STL
- link left_ring_PIP_Link: geometry collision mesh filename=meshes/hands/collision/left/left_ring_PIP_link.STL; collision mesh filename=meshes/hands/collision/left/left_ring_PIP_rubber_link.STL
- link left_thumb_CMP_Link: geometry collision mesh filename=meshes/hands/collision/left/left_thumb_CMP_link.STL; visual mesh filename=meshes/hands/visual/left/left_thumb_CMP_link.STL
- link left_thumb_CMR_Link: geometry collision mesh filename=meshes/hands/collision/left/cmr_v4_00.obj; collision mesh filename=meshes/hands/collision/left/cmr_v4_01.obj
- link left_thumb_DIP_Link: mass 0.01 -> 0.011; geometry collision mesh filename=meshes/hands/collision/left/left_thumb_DIP_link.STL; collision mesh filename=meshes/hands/collision/left/left_thumb_DIP_rubber_link.STL
- link left_thumb_MCP_Link: geometry collision mesh filename=meshes/hands/collision/left/left_thumb_MCP_link.STL; collision mesh filename=meshes/hands/collision/left/left_thumb_MCP_rubber_link.STL
- link left_thumb_PIP_Link: geometry collision mesh filename=meshes/hands/collision/left/left_thumb_PIP_link.STL; collision mesh filename=meshes/hands/collision/left/left_thumb_PIP_rubber_link.STL
- link right_hand_base_link: geometry collision mesh filename=meshes/hands/collision/right/right_hand_base_link.STL; collision mesh filename=meshes/hands/collision/right/right_palm_backtrim_v2.obj
- link right_index_DIP_Link: mass 0.010 -> 0.011; geometry collision mesh filename=meshes/hands/collision/right/right_index_DIP_link.STL; collision mesh filename=meshes/hands/collision/right/right_index_DIP_rubber_link.STL
- link right_index_MCP_Link: geometry collision mesh filename=meshes/hands/collision/right/right_index_MCP_link.STL; collision mesh filename=meshes/hands/collision/right/right_index_MCP_rubber_link.STL
- link right_index_MPR_Link: geometry collision mesh filename=meshes/hands/collision/right/right_index_MPR_link.STL; visual mesh filename=meshes/hands/visual/right/right_index_MPR_link.STL
- link right_index_PIP_Link: geometry collision mesh filename=meshes/hands/collision/right/right_index_PIP_link.STL; collision mesh filename=meshes/hands/collision/right/right_index_PIP_rubber_link.STL
- link right_little_DIP_Link: mass 0.010 -> 0.011; geometry collision mesh filename=meshes/hands/collision/right/right_little_DIP_link.STL; collision mesh filename=meshes/hands/collision/right/right_little_DIP_rubber_link.S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
- link right_little_MCP_Link: geometry collision mesh filename=meshes/hands/collision/right/right_little_MCP_link.STL; collision mesh filename=meshes/hands/collision/right/right_little_MCP_rubber_link.S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
- link right_little_MPR_Link: geometry collision mesh filename=meshes/hands/collision/right/right_little_MPR_link.STL; visual mesh filename=meshes/hands/visual/right/right_little_MPR_link.STL
- link right_little_PIP_Link: geometry collision mesh filename=meshes/hands/collision/right/right_little_PIP_link.STL; collision mesh filename=meshes/hands/collision/right/right_little_PIP_rubber_link.S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
- link right_middle_DIP_Link: mass 0.010 -> 0.011; geometry collision mesh filename=meshes/hands/collision/right/right_middle_DIP_link.STL; collision mesh filename=meshes/hands/collision/right/right_middle_DIP_rubber_link.S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
- link right_middle_MCP_Link: geometry collision mesh filename=meshes/hands/collision/right/right_middle_MCP_link.STL; collision mesh filename=meshes/hands/collision/right/right_middle_MCP_rubber_link.S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
- link right_middle_MPR_Link: geometry collision mesh filename=meshes/hands/collision/right/right_middle_MPR_link.STL; visual mesh filename=meshes/hands/visual/right/right_middle_MPR_link.STL
- link right_middle_PIP_Link: geometry collision mesh filename=meshes/hands/collision/right/right_middle_PIP_link.STL; collision mesh filename=meshes/hands/collision/right/right_middle_PIP_rubber_link.S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
- link right_ring_DIP_Link: mass 0.010 -> 0.011; geometry collision mesh filename=meshes/hands/collision/right/right_ring_DIP_link.STL; collision mesh filename=meshes/hands/collision/right/right_ring_DIP_rubber_link.STL
- link right_ring_MCP_Link: geometry collision mesh filename=meshes/hands/collision/right/right_ring_MCP_link.STL; collision mesh filename=meshes/hands/collision/right/right_ring_MCP_rubber_link.STL
- link right_ring_MPR_Link: geometry collision mesh filename=meshes/hands/collision/right/right_ring_MPR_link.STL; visual mesh filename=meshes/hands/visual/right/right_ring_MPR_link.STL
- link right_ring_PIP_Link: geometry collision mesh filename=meshes/hands/collision/right/right_ring_PIP_link.STL; collision mesh filename=meshes/hands/collision/right/right_ring_PIP_rubber_link.STL
- link right_thumb_CMP_Link: geometry collision mesh filename=meshes/hands/collision/right/right_thumb_CMP_link.STL; visual mesh filename=meshes/hands/visual/right/right_thumb_CMP_link.STL
- link right_thumb_CMR_Link: geometry collision mesh filename=meshes/hands/collision/right/cmr_v4_00.obj; collision mesh filename=meshes/hands/collision/right/cmr_v4_01.obj
- link right_thumb_DIP_Link: mass 0.010 -> 0.011; geometry collision mesh filename=meshes/hands/collision/right/right_thumb_DIP_link.STL; collision mesh filename=meshes/hands/collision/right/right_thumb_DIP_rubber_link.STL
- link right_thumb_MCP_Link: geometry collision mesh filename=meshes/hands/collision/right/right_thumb_MCP_link.STL; collision mesh filename=meshes/hands/collision/right/right_thumb_MCP_rubber_link.STL
- link right_thumb_PIP_Link: geometry collision mesh filename=meshes/hands/collision/right/right_thumb_PIP_link.STL; collision mesh filename=meshes/hands/collision/right/right_thumb_PIP_rubber_link.STL
Joints:
- removed joint left_palm_center
- removed joint right_palm_center
- joint left_index_DIP_joint: axis -0.05719 0.99648 0.061246 -> -0.057189678994825 0.996482943134821 0.061246099123401; limit lower=0 upper=1.4835 effort=0.35 velocity=6.28 -> lower=-0.322 upper=1.5978 effort=0 velocity=0; origin xyz=0.0013649 -0.0017312 0.029441 rpy=0 0 0 -> xyz=0.000140546972590664 -0.00180309239696645 0.0294678139594432 rpy=0 0 0
- joint left_index_MCP_joint: axis -0.05719 0.99648 0.061246 -> -0.0571896789948211 0.996482943134821 0.0612460991234106; limit lower=0 upper=1.4835 effort=0.35 velocity=6.28 -> lower=-0.0925 upper=1.583 effort=0 velocity=0; origin xyz=5.6148E-05 -0.00097833 0.01597 rpy=0 0 0 -> xyz=0.00185797304403404 -0.000875573004293424 0.0159806171918112 rpy=0 0 0
- joint left_index_MPR_joint: axis -0.99836 0.057297 0 -> 0.99835714347749 0.0572975918787191 0; limit lower=-0.2618 upper=0.2618 effort=0.35 velocity=6.28 -> lower=-0.1745 upper=0.5236 effort=0 velocity=0; origin xyz=-0.005442 -0.036871 0.097822 rpy=0 0 0 -> xyz=-0.00729368998766236 -0.036976393244618 0.0978111781534073 rpy=0 0 0
- joint left_index_PIP_joint: axis -0.05719 0.99648 0.061246 -> -0.0571896789948195 0.996482943134821 0.0612460991234103; limit lower=0 upper=1.4835 effort=0.35 velocity=6.28 -> lower=-0.1452 upper=1.6001 effort=0 velocity=0; origin xyz=0.00074519 -0.0028408 0.046916 rpy=0 0 0 -> xyz=0.000221764554223515 -0.00287108870207142 0.0469200922786802 rpy=0 0 0
- joint left_index_tip_joint: axis 0 0 0 -> (none)
- joint left_little_DIP_joint: axis 0.05719 0.99648 -0.061246 -> 0.0571896789757549 0.996482943138999 -0.0612460990732302; limit lower=0 upper=1.4835 effort=0.35 velocity=6.28 -> lower=-0.322 upper=1.5978 effort=0 velocity=0; origin xyz=0.0013649 0.0017312 0.029441 rpy=0 0 0 -> xyz=5.14511189704386E-05 0.00180820433011683 0.0294677909771798 rpy=0 0 0
- joint left_little_MCP_joint: axis 0.05719 0.99648 -0.061246 -> 0.0571896789757587 0.996482943139 -0.0612460990732217; limit lower=0 upper=1.4835 effort=0.35 velocity=6.28 -> lower=-0.0925 upper=1.583 effort=0 velocity=0; origin xyz=5.6148E-05 0.00097833 0.01597 rpy=0 0 0 -> xyz=0.00180966648562762 0.000878675609979826 0.0159859893072852 rpy=0 0 0
- joint left_little_MPR_joint: axis -0.99836 -0.057297 0 -> 0.998363207212642 -0.0571125018185487 0.00301141496872135; limit lower=-0.2618 upper=0.2618 effort=0.35 velocity=6.28 -> lower=-0.5236 upper=0.1745 effort=0 velocity=0; origin xyz=-0.0052198 0.036409 0.090532 rpy=0 0 0 -> xyz=-0.00702324534241969 0.0365118989929991 0.0905157916992934 rpy=0 0 0
- joint left_little_PIP_joint: axis 0.05719 0.99648 -0.061246 -> 0.0571896789757601 0.996482943138999 -0.0612460990732252; limit lower=0 upper=1.4835 effort=0.35 velocity=6.28 -> lower=-0.1452 upper=1.6001 effort=0 velocity=0; origin xyz=0.00074519 0.0028408 0.046916 rpy=0 0 0 -> xyz=7.99016655647876E-05 0.00287922592171121 0.0469200496920893 rpy=0 0 0
- joint left_little_tip_joint: axis 0 0 0 -> (none)
- joint left_middle_DIP_joint: axis -0.019101 0.99961 0.020433 -> -0.0191008584448469 0.999608742349558 0.0204332920745917; limit lower=0 upper=1.4835 effort=0.35 velocity=6.28 -> lower=-0.322 upper=1.5978 effort=0 velocity=0; origin xyz=0.0012747 -0.00057846 0.02949 rpy=0 0 0 -> xyz=0.000167169017596249 -0.000600164834043841 0.0295166870072403 rpy=0 0 0
- joint left_middle_MCP_joint: axis -0.019101 0.99961 0.020433 -> -0.0191008584448429 0.999608742349558 0.0204332920745991; limit lower=0 upper=1.4835 effort=0.35 velocity=6.28 -> lower=-0.0925 upper=1.583 effort=0 velocity=0; origin xyz=0 -0.00032687 0.015997 rpy=0 0 0 -> xyz=0.00187499938080231 -0.000291231468728885 0.0159999493531395 rpy=0 0 0
- joint left_middle_MPR_joint: axis -0.99982 0.019105 0 -> 0.999807814707845 0.019186925647608 -0.00402436744312752; limit lower=-0.2618 upper=0.2618 effort=0.35 velocity=6.28 -> lower=-0.3491 upper=0.4363 effort=0 velocity=0; origin xyz=-0.0060223 -0.012496 0.10793 rpy=0 0 0 -> xyz=-0.00794102299681282 -0.0125316383697077 0.107927151340908 rpy=0 0 0
- joint left_middle_PIP_joint: axis -0.019101 0.99961 0.020433 -> -0.0191008584448413 0.999608742349558 0.0204332920745958; limit lower=0 upper=1.4835 effort=0.35 velocity=6.28 -> lower=-0.1452 upper=1.6001 effort=0 velocity=0; origin xyz=0.00059944 -0.00094917 0.046994 rpy=0 0 0 -> xyz=0.000264150501422523 -0.00095565154131096 0.0469979185064267 rpy=0 0 0
- joint left_middle_tip_joint: axis 0 0 0 -> (none)
- joint left_ring_DIP_joint: axis 0.019101 0.99961 -0.020433 -> 0.0191008584234135 0.999608742351175 -0.0204332920154918; limit lower=0 upper=1.4835 effort=0.35 velocity=6.28 -> lower=-0.322 upper=1.5978 effort=0 velocity=0; origin xyz=0.0012747 0.00057846 0.02949 rpy=0 0 0 -> xyz=0.00011759316658046 0.00060111663666523 0.0295169067794739 rpy=0 0 0
- joint left_ring_MCP_joint: axis 0.019101 0.99961 -0.020433 -> 0.0191008584234173 0.999608742351176 -0.0204332920154781; limit lower=0 upper=1.4835 effort=0.35 velocity=6.28 -> lower=-0.0925 upper=1.583 effort=0 velocity=0; origin xyz=0 0.00032687 0.015997 rpy=0 0 0 -> xyz=0.00184812472405304 0.000291808729386601 0.0160030653444649 rpy=0 0 0
- joint left_ring_MPR_joint: axis -0.99982 -0.019105 0 -> 0.999813819455818 -0.0191527157615282 -0.00234518743967805; limit lower=-0.2618 upper=0.2618 effort=0.35 velocity=6.28 -> lower=-0.4363 upper=0.3491 effort=0 velocity=0; origin xyz=-0.0061966 0.012414 0.10384 rpy=0 0 0 -> xyz=-0.00808842265877729 0.0124508350538634 0.103836133387329 rpy=0 0 0
- joint left_ring_PIP_joint: axis 0.019101 0.99961 -0.020433 -> 0.0191008584234188 0.999608742351175 -0.0204332920154819; limit lower=0 upper=1.4835 effort=0.35 velocity=6.28 -> lower=-0.1452 upper=1.6001 effort=0 velocity=0; origin xyz=0.00059944 0.00094917 0.046994 rpy=0 0 0 -> xyz=0.000185213362502299 0.000957165097566284 0.0469982650773291 rpy=0 0 0
- joint left_ring_tip_joint: axis 0 0 0 -> (none)
- joint left_thumb_CMP_joint: limit lower=0 upper=1.9199 effort=0.35 velocity=6.28 -> lower=0 upper=1.92 effort=0 velocity=0; origin xyz=0.002 -0.0195 0.051993 rpy=0 0 0 -> xyz=0.00199783670091196 -0.0195358719276065 0.0520279736546372 rpy=0 0 0
- joint left_thumb_CMR_joint: axis 0 -1 0 -> 0 -0.999999985457346 0.000170544153169872; limit lower=0 upper=2.0071 effort=0.35 velocity=6.28 -> lower=-0.4224 upper=1.4277 effort=0 velocity=0; origin xyz=0 -0.0095 0 rpy=0 1.57 0 -> xyz=0 -0.0094641273542204 -3.19424156356996E-05 rpy=0 0 0
- joint left_thumb_DIP_joint: axis -1 0 0 -> -0.142628833818122 0.000168800639915566 0.989776230907788; limit lower=0 upper=1.4835 effort=0.35 velocity=6.28 -> lower=-0.16 upper=1.7616 effort=0 velocity=0; origin xyz=0 -0.031985 -0.00087263 rpy=0 0 0 -> xyz=0.000494631282394927 -0.0320003149826219 7.5667780971081E-05 rpy=0 0 0
- joint left_thumb_MCP_joint: axis -1 0 0 -> -0.142628833818122 0.000168800639916136 0.989776230907788; limit lower=0 upper=0.8727 effort=0.35 velocity=6.28 -> lower=-0.0845 upper=1.3292 effort=0 velocity=0; origin xyz=0 -0.0125 0 rpy=0 0 0 -> xyz=0 -0.0119999521610516 0 rpy=0 0 0
- joint left_thumb_PIP_joint: axis -1 0 0 -> -0.142628833818122 0.000168800639916073 0.989776230907788; limit lower=0 upper=1.4835 effort=0.35 velocity=6.28 -> lower=-0.2618 upper=1.5533 effort=0 velocity=0; origin xyz=0 -0.042087 -0.0013667 rpy=0 0 0 -> xyz=0 -0.0426092196906139 0 rpy=0 0 0
- joint left_thumb_tip_joint: axis 0 0 0 -> (none)
- joint right_index_DIP_joint: axis 0.05719 0.99648 -0.061255 -> 0.057189678994825 0.996482943134821 -0.061246099123401; limit lower=0 upper=1.4835 effort=0.35 velocity=6.28 -> lower=-0.322 upper=1.5978 effort=0 velocity=0; origin xyz=0.0013627 0.0017313 0.029441 rpy=0 0 0 -> xyz=0.000140546972590664 0.00180309239696645 0.0294678139594432 rpy=0 0 0
- joint right_index_MCP_joint: axis 0.05719 0.99648 -0.061246 -> 0.0571896789948211 0.996482943134821 -0.0612460991234106; limit lower=0 upper=1.4835 effort=0.35 velocity=6.28 -> lower=-0.0925 upper=1.583 effort=0 velocity=0; origin xyz=5.6148E-05 0.00097833 0.01597 rpy=0 0 0 -> xyz=0.00185797304403404 0.000875573004293424 0.0159806171918112 rpy=0 0 0
- joint right_index_MPR_joint: axis 0.99836 -0.057297 0 -> -0.99835714347749 0.0572975918787191 0; limit lower=-0.2618 upper=0.2618 effort=0.35 velocity=6.28 -> lower=-0.1745 upper=0.5236 effort=0 velocity=0; origin xyz=-0.005442 0.036871 0.097822 rpy=0 0 0 -> xyz=-0.00729368998766236 0.036976393244618 0.0978111781534073 rpy=0 0 0
- joint right_index_PIP_joint: axis 0.05719 0.99648 -0.061245 -> 0.0571896789948195 0.996482943134821 -0.0612460991234103; limit lower=0 upper=1.4835 effort=0.35 velocity=6.28 -> lower=-0.1452 upper=1.6001 effort=0 velocity=0; origin xyz=0.00074566 0.0028407 0.046916 rpy=0 0 0 -> xyz=0.000221764554223515 0.00287108870207142 0.0469200922786802 rpy=0 0 0
- joint right_index_tip_joint: axis 0 0 0 -> (none)
- joint right_little_DIP_joint: axis -0.057189 0.99648 0.061237 -> -0.0571896789757549 0.996482943138999 0.0612460990732302; limit lower=0 upper=1.4835 effort=0.35 velocity=6.28 -> lower=-0.322 upper=1.5978 effort=0 velocity=0; origin xyz=0.0013627 -0.0017313 0.029441 rpy=0 0 0 -> xyz=5.14511189704386E-05 -0.00180820433011683 0.0294677909771798 rpy=0 0 0
- joint right_little_MCP_joint: axis -0.05719 0.99648 0.061246 -> -0.0571896789757587 0.996482943139 0.0612460990732217; limit lower=0 upper=1.4835 effort=0.35 velocity=6.28 -> lower=-0.0925 upper=1.583 effort=0 velocity=0; origin xyz=5.6148E-05 -0.00097833 0.01597 rpy=0 0 0 -> xyz=0.00180966648562762 -0.000878675609979826 0.0159859893072852 rpy=0 0 0
- joint right_little_MPR_joint: axis 0.99836 0.057297 0 -> -0.998363207212642 -0.0571125018185487 -0.00301141496872135; limit lower=-0.2618 upper=0.2618 effort=0.35 velocity=6.28 -> lower=-0.5236 upper=0.1745 effort=0 velocity=0; origin xyz=-0.0052697 -0.036412 0.090532 rpy=0 0 0 -> xyz=-0.00702324534241969 -0.0365118989929991 0.0905157916992934 rpy=0 0 0
- joint right_little_PIP_joint: axis -0.05719 0.99648 0.061247 -> -0.0571896789757601 0.996482943138999 0.0612460990732252; limit lower=0 upper=1.4835 effort=0.35 velocity=6.28 -> lower=-0.1452 upper=1.6001 effort=0 velocity=0; origin xyz=0.00079558 -0.0028379 0.046916 rpy=0 0 0 -> xyz=7.99016655647876E-05 -0.00287922592171121 0.0469200496920893 rpy=0 0 0
- joint right_little_tip_joint: axis 0 0 0 -> (none)
- joint right_middle_DIP_joint: axis 0.019101 0.99961 -0.020443 -> 0.0191008584448469 0.999608742349558 -0.0204332920745917; limit lower=0 upper=1.4835 effort=0.35 velocity=6.28 -> lower=-0.322 upper=1.5978 effort=0 velocity=0; origin xyz=0.0012725 0.00057847 0.02949 rpy=0 0 0 -> xyz=0.000167169017596249 0.000600164834043841 0.0295166870072403 rpy=0 0 0
- joint right_middle_MCP_joint: axis 0.019101 0.99961 -0.020433 -> 0.0191008584448429 0.999608742349558 -0.0204332920745991; limit lower=0 upper=1.4835 effort=0.35 velocity=6.28 -> lower=-0.0925 upper=1.583 effort=0 velocity=0; origin xyz=0 0.00032687 0.015997 rpy=0 0 0 -> xyz=0.00187499938080231 0.000291231468728885 0.0159999493531395 rpy=0 0 0
- joint right_middle_MPR_joint: axis 0.99982 -0.019105 0 -> -0.999807814707845 0.019186925647608 0.00402436744312752; limit lower=-0.2618 upper=0.2618 effort=0.35 velocity=6.28 -> lower=-0.3491 upper=0.4363 effort=0 velocity=0; origin xyz=-0.0060223 0.012496 0.10793 rpy=0 0 0 -> xyz=-0.00794102299681282 0.0125316383697077 0.107927151340908 rpy=0 0 0
- joint right_middle_PIP_joint: axis 0.019101 0.99961 -0.020432 -> 0.0191008584448413 0.999608742349558 -0.0204332920745958; limit lower=0 upper=1.4835 effort=0.35 velocity=6.28 -> lower=-0.1452 upper=1.6001 effort=0 velocity=0; origin xyz=0.00059991 0.00094912 0.046994 rpy=0 0 0 -> xyz=0.000264150501422523 0.00095565154131096 0.0469979185064267 rpy=0 0 0
- joint right_middle_tip_joint: axis 0 0 0 -> (none)
- joint right_ring_DIP_joint: axis -0.019101 0.99961 0.020424 -> -0.0191008584234135 0.999608742351175 0.0204332920154918; limit lower=0 upper=1.4835 effort=0.35 velocity=6.28 -> lower=-0.322 upper=1.5978 effort=0 velocity=0; origin xyz=0.0012725 -0.00057823 0.02949 rpy=0 0 0 -> xyz=0.00011759316658046 -0.00060111663666523 0.0295169067794739 rpy=0 0 0
- joint right_ring_MCP_joint: axis -0.019101 0.99961 0.020433 -> -0.0191008584234173 0.999608742351176 0.0204332920154781; limit lower=0 upper=1.4835 effort=0.35 velocity=6.28 -> lower=-0.0925 upper=1.583 effort=0 velocity=0; origin xyz=0 -0.00032687 0.015997 rpy=0 0 0 -> xyz=0.00184812472405304 -0.000291808729386601 0.0160030653444649 rpy=0 0 0
- joint right_ring_MPR_joint: axis 0.99982 0.019105 0 -> -0.999813819455818 -0.0191527157615282 0.00234518743967805; limit lower=-0.2618 upper=0.2618 effort=0.35 velocity=6.28 -> lower=-0.4363 upper=0.3491 effort=0 velocity=0; origin xyz=-0.0062466 -0.012415 0.10384 rpy=0 0 0 -> xyz=-0.00808842265877729 -0.0124508350538634 0.103836133387329 rpy=0 0 0
- joint right_ring_PIP_joint: axis -0.019101 0.99961 0.020434 -> -0.0191008584234188 0.999608742351175 0.0204332920154819; limit lower=0 upper=1.4835 effort=0.35 velocity=6.28 -> lower=-0.1452 upper=1.6001 effort=0 velocity=0; origin xyz=0.0006499 -0.00094821 0.046994 rpy=0 0 0 -> xyz=0.000185213362502299 -0.000957165097566284 0.0469982650773291 rpy=0 0 0
- joint right_ring_tip_joint: axis 0 0 0 -> (none)
- joint right_thumb_CMP_joint: limit lower=0 upper=1.9199 effort=0.35 velocity=6.28 -> lower=0 upper=1.92 effort=0 velocity=0; origin xyz=0.002 0.0195 0.051993 rpy=0 0 0 -> xyz=0.00199783670091196 0.0195358719276065 0.0520279736546372 rpy=0 0 0
- joint right_thumb_CMR_joint: axis 0 -1 0 -> 0 -0.999999985457346 -0.000170544153169872; limit lower=0 upper=2.0071 effort=0.35 velocity=6.28 -> lower=-0.4224 upper=1.4277 effort=0 velocity=0; origin xyz=0 0.0095 0 rpy=0 1.57 0 -> xyz=0 0.0094641273542204 -3.19424156356996E-05 rpy=0 0 0
- joint right_thumb_DIP_joint: axis 1 0 0 -> 0.142628833818122 0.000168800639915566 -0.989776230907788; limit lower=0 upper=1.4835 effort=0.35 velocity=6.28 -> lower=-0.16 upper=1.7616 effort=0 velocity=0; origin xyz=0.000125 0.032 -0.00052077 rpy=0 0 0 -> xyz=0.000494631282394927 0.0320003149826219 7.5667780971081E-05 rpy=0 0 0
- joint right_thumb_MCP_joint: axis 1 0 0 -> 0.142628833818122 0.000168800639916136 -0.989776230907788; limit lower=0 upper=0.8727 effort=0.35 velocity=6.28 -> lower=-0.0845 upper=1.3292 effort=0 velocity=0; origin xyz=0 0.0125 0 rpy=0 0 0 -> xyz=0 0.0119999521610516 0 rpy=0 0 0
- joint right_thumb_PIP_joint: axis 1 0 0 -> 0.142628833818122 0.000168800639916073 -0.989776230907788; limit lower=0 upper=1.4835 effort=0.35 velocity=6.28 -> lower=-0.2618 upper=1.5533 effort=0 velocity=0; origin xyz=0.0001 0.042087 -0.0013667 rpy=0 0 0 -> xyz=0 0.0426092196906139 0 rpy=0 0 0
- joint right_thumb_tip_joint: axis 0 0 0 -> (none)
