Commit message: Replace training URDF with supplied reduced28 articulation

File: assets/assembly_rl_convex.urdf (robot description, URDF)
Before this commit: robot tron2_dach_revo3_d455_supplied_step_brackets, 116 links, 115 joints
Links:
- removed link base_2_Link
- removed link base_3_Link
- removed link base_imu
- removed link d435_Link
- removed link d435_optical_frame
- removed link elbow_L_Link
- removed link head_base_Link
- removed link head_camera_accel_frame
- removed link head_camera_accel_optical_frame
- removed link head_camera_bottom_screw_frame
- removed link head_camera_color_frame
- removed link head_camera_color_optical_frame
- removed link head_camera_depth_frame
- removed link head_camera_depth_optical_frame
- removed link head_camera_gyro_frame
- removed link head_camera_gyro_optical_frame
- removed link head_camera_imu_optical_frame
- removed link head_camera_infra1_frame
- removed link head_camera_infra1_optical_frame
- removed link head_camera_infra2_frame
- removed link head_camera_infra2_optical_frame
- removed link head_camera_link
- removed link head_camera_mount_frame
- removed link head_pitch_Link
- removed link head_yaw_Link
- removed link left_adapter_link
- removed link left_hand_base_link
- removed link left_index_DIP_Link
- removed link left_index_MCP_Link
- removed link left_index_MPR_Link
- removed link left_index_PIP_Link
- removed link left_index_tip_Link
- removed link left_little_DIP_Link
- removed link left_little_MCP_Link
- removed link left_little_MPR_Link
- removed link left_little_PIP_Link
- removed link left_little_tip_Link
- removed link left_middle_DIP_Link
- removed link left_middle_MCP_Link
- removed link left_middle_MPR_Link
- removed link left_middle_PIP_Link
- removed link left_middle_tip_Link
- removed link left_palm
- removed link left_ring_DIP_Link
- removed link left_ring_MCP_Link
- removed link left_ring_MPR_Link
- removed link left_ring_PIP_Link
- removed link left_ring_tip_Link
- removed link left_thumb_CMP_Link
- removed link left_thumb_CMR_Link
- removed link left_thumb_DIP_Link
- removed link left_thumb_MCP_Link
- removed link left_thumb_PIP_Link
- removed link left_thumb_tip_Link
- removed link left_wrist_camera_bottom_screw_frame
- removed link left_wrist_camera_color_frame
- removed link left_wrist_camera_color_optical_frame
- removed link left_wrist_camera_depth_frame
- removed link left_wrist_camera_depth_optical_frame
- removed link left_wrist_camera_link
- removed link left_wrist_camera_mount_frame
- removed link left_wrist_camera_plate_frame
- removed link left_wrist_camera_rod_end_frame
- removed link proximal_pitch_L_Link
- removed link proximal_roll_L_Link
- removed link proximal_yaw_L_Link
- removed link right_wrist_camera_bottom_screw_frame
- removed link right_wrist_camera_color_frame
- removed link right_wrist_camera_color_optical_frame
- removed link right_wrist_camera_depth_frame
- removed link right_wrist_camera_depth_optical_frame
- removed link right_wrist_camera_link
- removed link right_wrist_camera_mount_frame
- removed link right_wrist_camera_plate_frame
- removed link right_wrist_camera_rod_end_frame
- removed link wrist_pitch_L_Link
- removed link wrist_roll_L_Link
- removed link wrist_yaw_L_Link
- link base_Link: mass 12.57 -> 53.4949868056; geometry collision mesh filename=meshes/boundaryfix_exact/collision_2352ac2b3de24d8b94aa3985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; visual box size=0.005 0.005 0.005
- link elbow_R_Link: geometry collision mesh filename=meshes/boundaryfix_exact/c931c244ccb1b6ef6a694ca03f9b7fef64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; visual mesh filename=meshes/tron2/elbow_R_Link.STL
- link proximal_pitch_R_Link: geometry collision mesh filename=meshes/boundaryfix_exact/collision_18d038d6ab285f6ed9caa84c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; visual mesh filename=meshes/tron2/proximal_pitch_R_Link.STL
- link proximal_roll_R_Link: geometry collision mesh filename=meshes/boundaryfix_exact/collision_399f3fcd0e8392e9d1ef8366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; visual mesh filename=meshes/tron2/proximal_roll_R_Link.STL
- link proximal_yaw_R_Link: geometry collision mesh filename=meshes/boundaryfix_exact/collision_697b41afc439a30e0fb51bfc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; visual cylinder length=0.010 radius=0.054
- link right_adapter_link: mass 0.103444531962598 -> 0.103444531963; geometry collision mesh filename=meshes/right_adapter_single_convex.obj; visual mesh filename=meshes/adapter_v2/right/adapter_right_v2_visual.stl
- link right_hand_base_link: geometry collision mesh filename=meshes/right_palm_single_convex.obj; visual mesh filename=meshes/revo3/hands/visual/right/revo3__hands__visual__right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
- link right_index_DIP_Link: mass 0.010 -> 0.01; geometry collision mesh filename=meshes/boundaryfix_exact/eac2fb6f67be2bf45c8847b7b228a01147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; visual mesh filename=meshes/revo3/hands/visual/right/revo3__hands__visual__right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
- link right_index_MCP_Link: geometry collision mesh filename=meshes/boundaryfix_exact/collision_84a94c7c4910d28b6cd335b0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; visual mesh filename=meshes/revo3/hands/visual/right/revo3__hands__visual__right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
- link right_index_MPR_Link: geometry collision mesh filename=meshes/boundaryfix_exact/dd474f932d933c7f19b1427ab848dba39d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; visual mesh filename=meshes/revo3/hands/visual/right/revo3__hands__visual__right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
- link right_index_PIP_Link: geometry collision mesh filename=meshes/boundaryfix_exact/cd4974214ec991982752c834207b5a55e8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; visual mesh filename=meshes/revo3/hands/visual/right/revo3__hands__visual__right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
- link right_little_DIP_Link: mass 0.010 -> 0.01; geometry collision mesh filename=meshes/boundaryfix_exact/collision_424fb5d42fe910674e2070a3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; visual mesh filename=meshes/revo3/hands/visual/right/revo3__hands__visual__right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
- link right_little_MCP_Link: geometry collision mesh filename=meshes/boundaryfix_exact/collision_444b3d2be3ad94f1e91f12a4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; visual mesh filename=meshes/revo3/hands/visual/right/revo3__hands__visual__right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
- link right_little_MPR_Link: geometry collision mesh filename=meshes/boundaryfix_exact/f0f14494856f0b384b36ee3961d8f0e1a6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; visual mesh filename=meshes/revo3/hands/visual/right/revo3__hands__visual__right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
- link right_little_PIP_Link: geometry collision mesh filename=meshes/boundaryfix_exact/collision_0b9fcebfd5221679b6614967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; visual mesh filename=meshes/revo3/hands/visual/right/revo3__hands__visual__right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
- link right_middle_DIP_Link: mass 0.010 -> 0.01; geometry collision mesh filename=meshes/boundaryfix_exact/collision_48f25a0c8992909af1db8385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; visual mesh filename=meshes/revo3/hands/visual/right/revo3__hands__visual__right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
- link right_middle_MCP_Link: geometry collision mesh filename=meshes/boundaryfix_exact/c61f048e7e643dc2eadfc6b32a4c19f0dd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; visual mesh filename=meshes/revo3/hands/visual/right/revo3__hands__visual__right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
- link right_middle_MPR_Link: geometry collision mesh filename=meshes/boundaryfix_exact/collision_779f45b6eaa9078ee49cd641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; visual mesh filename=meshes/revo3/hands/visual/right/revo3__hands__visual__right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
- link right_middle_PIP_Link: geometry collision mesh filename=meshes/boundaryfix_exact/collision_01c7f36fb939a05d47f7330d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; visual mesh filename=meshes/revo3/hands/visual/right/revo3__hands__visual__right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
- link right_ring_DIP_Link: mass 0.010 -> 0.01; geometry collision mesh filename=meshes/boundaryfix_exact/f09b2b654f0ce9c206e33660cdf8adcd41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; visual mesh filename=meshes/revo3/hands/visual/right/revo3__hands__visual__right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
- link right_ring_MCP_Link: geometry collision mesh filename=meshes/boundaryfix_exact/collision_8b8a22e190e5ed119e859726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; visual mesh filename=meshes/revo3/hands/visual/right/revo3__hands__visual__right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
- link right_ring_MPR_Link: geometry collision mesh filename=meshes/boundaryfix_exact/collision_6d5130521d5db18a9b323fde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; visual mesh filename=meshes/revo3/hands/visual/right/revo3__hands__visual__right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
- link right_ring_PIP_Link: geometry collision mesh filename=meshes/boundaryfix_exact/collision_4ecfdad5c0c16b4baa803d12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; visual mesh filename=meshes/revo3/hands/visual/right/revo3__hands__visual__right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
- link right_thumb_CMP_Link: geometry collision mesh filename=meshes/boundaryfix_exact/collision_5f337ce59f54aad60fc17839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; visual mesh filename=meshes/revo3/hands/visual/right/revo3__hands__visual__right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
- link right_thumb_CMR_Link: geometry collision mesh filename=meshes/boundaryfix_exact/collision_68413dc1bf233abbacc1bbd3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; visual mesh filename=meshes/revo3/hands/visual/right/revo3__hands__visual__right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
- link right_thumb_DIP_Link: mass 0.010 -> 0.01; geometry collision mesh filename=meshes/boundaryfix_exact/collision_9c29beced59e6cbdc686a68c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; visual mesh filename=meshes/revo3/hands/visual/right/revo3__hands__visual__right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
- link right_thumb_MCP_Link: geometry collision mesh filename=meshes/boundaryfix_exact/ebef9bc72a318403c46f3907fd35b21afd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; visual mesh filename=meshes/revo3/hands/visual/right/revo3__hands__visual__right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
- link right_thumb_PIP_Link: geometry collision mesh filename=meshes/boundaryfix_exact/collision_4eab982141d3f32b09b16a74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; visual mesh filename=meshes/revo3/hands/visual/right/revo3__hands__visual__right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
- link wrist_pitch_R_Link: geometry collision mesh filename=meshes/boundaryfix_exact/collision_9a43ecc1054746888f535f49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; visual mesh filename=meshes/tron2/wrist_pitch_R_Link.STL
- link wrist_roll_R_Link: mass 0.24 -> 0.264939446617; geometry collision mesh filename=meshes/boundaryfix_exact/collision_7f750db7fdcfd687d4076675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; visual mesh filename=meshes/cameras/d405_visual_m.stl
- link wrist_yaw_R_Link: geometry collision mesh filename=meshes/boundaryfix_exact/ae4e19d5bdef3680d3e0ea14c38aaf667e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; visual cylinder length=0.008 radius=0.043
Joints:
- removed joint base_2_Joint
- removed joint base_3_Joint
- removed joint base_imu_Joint
- removed joint d435_Joint
- removed joint d435_optical_Joint
- removed joint elbow_L_Joint
- removed joint head_base_Joint
- removed joint head_camera_accel_joint
- removed joint head_camera_accel_optical_joint
- removed joint head_camera_color_joint
- removed joint head_camera_color_optical_joint
- removed joint head_camera_depth_joint
- removed joint head_camera_depth_optical_joint
- removed joint head_camera_gyro_joint
- removed joint head_camera_gyro_optical_joint
- removed joint head_camera_imu_optical_joint
- removed joint head_camera_infra1_joint
- removed joint head_camera_infra1_optical_joint
- removed joint head_camera_infra2_joint
- removed joint head_camera_infra2_optical_joint
- removed joint head_camera_link_joint
- removed joint head_camera_mount_joint
- removed joint head_camera_reference_joint
- removed joint head_pitch_Joint
- removed joint head_yaw_Joint
- removed joint left_adapter_mount
- removed joint left_hand_base_joint
- removed joint left_index_DIP_joint
- removed joint left_index_MCP_joint
- removed joint left_index_MPR_joint
- removed joint left_index_PIP_joint
- removed joint left_index_tip_joint
- removed joint left_little_DIP_joint
- removed joint left_little_MCP_joint
- removed joint left_little_MPR_joint
- removed joint left_little_PIP_joint
- removed joint left_little_tip_joint
- removed joint left_middle_DIP_joint
- removed joint left_middle_MCP_joint
- removed joint left_middle_MPR_joint
- removed joint left_middle_PIP_joint
- removed joint left_middle_tip_joint
- removed joint left_palm_center
- removed joint left_ring_DIP_joint
- removed joint left_ring_MCP_joint
- removed joint left_ring_MPR_joint
- removed joint left_ring_PIP_joint
- removed joint left_ring_tip_joint
- removed joint left_thumb_CMP_joint
- removed joint left_thumb_CMR_joint
- removed joint left_thumb_DIP_joint
- removed joint left_thumb_MCP_joint
- removed joint left_thumb_PIP_joint
- removed joint left_thumb_tip_joint
- removed joint left_wrist_camera_color_joint
- removed joint left_wrist_camera_color_optical_joint
- removed joint left_wrist_camera_depth_joint
- removed joint left_wrist_camera_depth_optical_joint
- removed joint left_wrist_camera_extension_joint
- removed joint left_wrist_camera_link_joint
- removed joint left_wrist_camera_mount_joint
- removed joint left_wrist_camera_plate_joint
- removed joint left_wrist_camera_reference_joint
- removed joint proximal_pitch_L_Joint
- removed joint proximal_roll_L_Joint
- removed joint proximal_yaw_L_Joint
- removed joint right_wrist_camera_color_joint
- removed joint right_wrist_camera_color_optical_joint
- removed joint right_wrist_camera_depth_joint
- removed joint right_wrist_camera_depth_optical_joint
- removed joint right_wrist_camera_extension_joint
- removed joint right_wrist_camera_link_joint
- removed joint right_wrist_camera_mount_joint
- removed joint right_wrist_camera_plate_joint
- removed joint right_wrist_camera_reference_joint
- removed joint wrist_pitch_L_Joint
- removed joint wrist_roll_L_Joint
- removed joint wrist_yaw_L_Joint

Commit message: Publish current physicsfix training URDF and synchronized asset docs

File: assets/assembly_rl_convex.urdf (robot description, URDF)
Before this commit: robot tron2_dach_revo3_d455_supplied_step_brackets, 38 links, 37 joints
Links:
- link right_hand_base_link: geometry collision mesh filename=meshes/boundaryfix_exact/a4023ceff84d9f0ad52b57589535087596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; collision mesh filename=meshes/boundaryfix_exact/a8da7d01b52a7d7c1852e4f3ddec632b68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
- link right_index_tip_Link: mass None -> 0.001
- link right_little_tip_Link: mass None -> 0.001
- link right_middle_tip_Link: mass None -> 0.001
- link right_ring_tip_Link: mass None -> 0.001
- link right_thumb_tip_Link: mass None -> 0.001

Commit message: Replace reduced training URDF with validated 58-collision model
Preserve official Revo3 kinematics, inertias, mount transforms and DIP contact geometry. Package same-link convex meshes, hash manifests and paired documentation; verify 20 asset tests and the current contact-v5 trajectory binding.

File: assets/assembly_rl_convex.urdf (robot description, URDF)
Before this commit: robot tron2_dach_revo3_d455_supplied_step_brackets, 37 links, 36 joints
Links:
- link right_hand_base_link: geometry collision mesh filename=collision58_meshes/right_hand_base_link_01.obj; collision mesh filename=meshes/hands/collision/right/right_hand_base_link.STL
- link right_index_MCP_Link: geometry collision mesh filename=collision58_meshes/right_index_MCP_Link_01.obj; collision mesh filename=meshes/hands/collision/right/right_index_MCP_link.STL
- link right_index_PIP_Link: geometry collision mesh filename=collision58_meshes/right_index_PIP_Link_00.obj; visual mesh filename=meshes/hands/visual/right/right_index_PIP_link.STL
- link right_little_MCP_Link: geometry collision mesh filename=collision58_meshes/right_little_MCP_Link_00.obj; visual mesh filename=meshes/hands/visual/right/right_little_MCP_link.STL
- link right_little_PIP_Link: geometry collision mesh filename=collision58_meshes/right_little_PIP_Link_00.obj; visual mesh filename=meshes/hands/visual/right/right_little_PIP_link.STL
- link right_middle_MCP_Link: geometry collision mesh filename=collision58_meshes/right_middle_MCP_Link_01.obj; collision mesh filename=meshes/hands/collision/right/right_middle_MCP_link.STL
- link right_middle_PIP_Link: geometry collision mesh filename=collision58_meshes/right_middle_PIP_Link_00.obj; visual mesh filename=meshes/hands/visual/right/right_middle_PIP_link.STL
- link right_ring_MCP_Link: geometry collision mesh filename=collision58_meshes/right_ring_MCP_Link_00.obj; visual mesh filename=meshes/hands/visual/right/right_ring_MCP_link.STL
- link right_ring_PIP_Link: geometry collision mesh filename=collision58_meshes/right_ring_PIP_Link_00.obj; visual mesh filename=meshes/hands/visual/right/right_ring_PIP_link.STL
- link right_thumb_CMR_Link: geometry collision mesh filename=collision58_meshes/right_thumb_CMR_Link_02.obj; collision mesh filename=collision58_meshes/right_thumb_CMR_Link_03.obj
- link right_thumb_MCP_Link: geometry collision mesh filename=collision58_meshes/right_thumb_MCP_Link_00.obj; visual mesh filename=meshes/hands/visual/right/right_thumb_MCP_link.STL
- link right_thumb_PIP_Link: geometry collision mesh filename=collision58_meshes/right_thumb_PIP_Link_00.obj; visual mesh filename=meshes/hands/visual/right/right_thumb_PIP_link.STL
